Commit message: Update vlp16.xacro

File: src/learnbotic/learnbotic_description/urdf/vlp16.xacro (robot description, xacro)
@@ -33,6 +33,4 @@
       </sensor>
     </gazebo>
-    <link name="base_sensor">
-    </link>
     <link name="sensor">
       <inertial>
@@ -53,8 +51,3 @@
       </visual>
     </link>
-    <joint name="base_to_sensor" type="fixed">
-      <parent link="base_sensor"/>
-      <child link="sensor"/>
-      <origin rpy="0 0 0" xyz="0.0 0.0 0.0"/>
-    </joint>
   </robot>
