Commit message: Update model.urdf

File: src/learnbotic/learnbotic_description/urdf/model.urdf (robot description, URDF)
Before this commit: robot learnbotic, 7 links, 8 joints
Joints:
- joint lidar: axis (none) -> 0 0 1; child base_sensor -> sensor; limit (none) -> lower=-1.79769e+308 upper=1.79769e+308 effort=-1.0 velocity=1.0; type fixed -> revolute

Commit message: add plugin giro

File: src/learnbotic/learnbotic_description/urdf/model.urdf (robot description, URDF)
Before this commit: robot learnbotic, 7 links, 8 joints
Joints:
- joint lidar: axis 0 0 1 -> (none); child sensor -> sensor1; limit lower=-1.79769e+308 upper=1.79769e+308 effort=-1.0 velocity=1.0 -> (none); origin xyz=0 0.049 0 rpy=1.571 0 0 -> xyz=0 0.049 0 rpy=-1.571 0 0; type revolute -> fixed

File: src/learnbotic/learnbotic_description/urdf/vlp16.xacro (robot description, xacro)
@@ -1,4 +1,4 @@
 <?xml version="1.0" ?>
-  <robot name="vlp-16" xmlns:xacro="http://ros.org/wiki/xacro">
+  <robot name="vlp16" xmlns:xacro="http://ros.org/wiki/xacro">
     <gazebo reference="sensor">
       <sensor type="ray" name="vlp">
@@ -14,10 +14,16 @@
           </noise>
           <scan>
-            <horizontal>
+            <!-- <horizontal>
               <samples>360</samples>
               <resolution>1</resolution>
+              <min_angle>-3.14</min_angle>
+              <max_angle>3.14</max_angle>
+            </horizontal> -->
+            <vertical>
+              <samples>16</samples>
+              <resolution>1</resolution>
               <min_angle>0</min_angle>
-              <max_angle>6.28</max_angle>
-            </horizontal>
+              <max_angle>0.18</max_angle>
+            </vertical>
           </scan>
           <range>
@@ -27,5 +33,8 @@
           </range>
         </ray>
-        <plugin name="gazebo_ros_laser_controller" filename="libgazebo_ros_laser.so">
+          <plugin name="velodyne_control" filename="libvelodybe_plugin.so">
+            <robotNamespace>/</robotNamespace>
+          </plugin>
+          <plugin name="gazebo_ros_laser_controller" filename="libgazebo_ros_velodyne_laser.so">
           <topicName>/diff/laser/scan</topicName>
           <frameName>sensor</frameName>
@@ -33,5 +42,5 @@
       </sensor>
     </gazebo>
-    <link name="sensor">
+    <link name="sensor1">
       <inertial>
         <origin rpy="0 0 0" xyz="0 0 0"/>
@@ -39,5 +48,5 @@
         <inertia ixx="0.000909131" iyy="0.000909131" izz="0.001107105" ixy="0" ixz="0" iyz="0"/>
       </inertial>
-      <collision>
+       <collision>
         <origin rpy="0 0 0" xyz="0 0 0"/>
         <geometry>
@@ -51,3 +60,23 @@
       </visual>
     </link>
+    <link name="sensor">
+      <inertial>
+        <origin rpy="0 0 0" xyz="0 0 0"/>
+        <mass value ="0.05"/>
+        <inertia ixx="0.000909131" iyy="0.000909131" izz="0.001107105" ixy="0" ixz="0" iyz="0"/>
+      </inertial>
+    </link>
+    <joint name="giro" type="revolute">
+      <parent link="sensor1"/>
+      <child link="sensor"/>
+      <origin rpy="0 0 0" xyz="0 0 0"/>
+      <axis xyz="0 0 1"/>
+      <limit effort="-1" lower="-1.79769e+308" upper="1.79769e+308" velocity="100"/>
+    </joint>
+  <gazebo>
+    <plugin name="velodyne_control" filename="libvelodyne_plugin.so">
+      <test>giro</test>
+      <velocity>50</velocity>
+    </plugin>
+  </gazebo>
   </robot>
